Commit message: tibia sidedness fix

File: urdf/leg.xacro (robot description, xacro)
@@ -168,7 +168,7 @@
   <link name="${name}_tibia_link">
     <visual>
-      <origin rpy="0 0 ${pi}" xyz="0.007 0 -0.03"/>
+      <origin rpy="0 0 0" xyz="0.007 0 -0.03"/>
       <geometry>
-        <mesh filename="package://open_critter/meshes/collada/tibia_front.dae"/>
+        <mesh filename="package://open_critter/meshes/collada/tibia_rear.dae"/>
       </geometry>
     </visual>

Commit message: description launch

File: urdf/leg.xacro (robot description, xacro)
@@ -23,4 +23,15 @@
       <axis xyz="0 0 1"/>
     </joint>
+    <transmission name="${name}_coxa_servo_transmission">
+        <type>transmission_interface/SimpleTransmission</type>
+        <joint name="${name}_coxa_servo_joint">
+            <hardwareInterface>hardware_interface/PositionJointInterface</hardwareInterface>
+        </joint>
+        <actuator name="${name}_coxa_servo_actuator">
+            <hardwareInterface>hardware_interface/PositionJointInterface</hardwareInterface>
+            <mechanicalReduction>1</mechanicalReduction>
+            <motorTorqueConstant>1</motorTorqueConstant>
+        </actuator>
+    </transmission>
     <link name="${name}_coxa_link">
       <visual>
@@ -51,4 +62,15 @@
       <axis xyz="1 0 0"/>
     </joint>
+    <transmission name="${name}_femur_servo_transmission">
+        <type>transmission_interface/SimpleTransmission</type>
+        <joint name="${name}_femur_servo_joint">
+            <hardwareInterface>hardware_interface/PositionJointInterface</hardwareInterface>
+        </joint>
+        <actuator name="${name}_femur_servo_actuator">
+            <hardwareInterface>hardware_interface/PositionJointInterface</hardwareInterface>
+            <mechanicalReduction>1</mechanicalReduction>
+            <motorTorqueConstant>1</motorTorqueConstant>
+        </actuator>
+    </transmission>
     <link name="${name}_femur_link">
       <visual>
@@ -66,4 +88,15 @@
       <axis xyz="1 0 0"/>
     </joint>
+    <transmission name="${name}_tibia_servo_transmission">
+        <type>transmission_interface/SimpleTransmission</type>
+        <joint name="${name}_tibia_servo_joint">
+            <hardwareInterface>hardware_interface/PositionJointInterface</hardwareInterface>
+        </joint>
+        <actuator name="${name}_tibia_servo_actuator">
+            <hardwareInterface>hardware_interface/PositionJointInterface</hardwareInterface>
+            <mechanicalReduction>1</mechanicalReduction>
+            <motorTorqueConstant>1</motorTorqueConstant>
+        </actuator>
+    </transmission>
     <link name="${name}_tibia_servo">
       <visual>
@@ -110,4 +143,15 @@
     <axis xyz="0 0 1"/>
   </joint>
+  <transmission name="${name}_coxa_servo_transmission">
+      <type>transmission_interface/SimpleTransmission</type>
+      <joint name="${name}_coxa_servo_joint">
+          <hardwareInterface>hardware_interface/PositionJointInterface</hardwareInterface>
+      </joint>
+      <actuator name="${name}_coxa_servo_actuator">
+          <hardwareInterface>hardware_interface/PositionJointInterface</hardwareInterface>
+          <mechanicalReduction>1</mechanicalReduction>
+          <motorTorqueConstant>1</motorTorqueConstant>
+      </actuator>
+  </transmission>
   <link name="${name}_coxa_link">
     <visual>
@@ -138,4 +182,15 @@
     <axis xyz="1 0 0"/>
   </joint>
+  <transmission name="${name}_femur_servo_transmission">
+      <type>transmission_interface/SimpleTransmission</type>
+      <joint name="${name}_femur_servo_joint">
+          <hardwareInterface>hardware_interface/PositionJointInterface</hardwareInterface>
+      </joint>
+      <actuator name="${name}_femur_servo_actuator">
+          <hardwareInterface>hardware_interface/PositionJointInterface</hardwareInterface>
+          <mechanicalReduction>1</mechanicalReduction>
+          <motorTorqueConstant>1</motorTorqueConstant>
+      </actuator>
+  </transmission>
   <link name="${name}_femur_link">
     <visual>
@@ -153,4 +208,15 @@
     <axis xyz="1 0 0"/>
   </joint>
+  <transmission name="${name}_tibia_servo_transmission">
+      <type>transmission_interface/SimpleTransmission</type>
+      <joint name="${name}_tibia_servo_joint">
+          <hardwareInterface>hardware_interface/PositionJointInterface</hardwareInterface>
+      </joint>
+      <actuator name="${name}_tibia_servo_actuator">
+          <hardwareInterface>hardware_interface/PositionJointInterface</hardwareInterface>
+          <mechanicalReduction>1</mechanicalReduction>
+          <motorTorqueConstant>1</motorTorqueConstant>
+      </actuator>
+  </transmission>
   <link name="${name}_tibia_servo">
     <visual>

Commit message: somewhat okayish sim

File: urdf/leg.xacro (robot description, xacro)
@@ -56,5 +56,5 @@
     <child link="${name}_coxa_link"/>
     <origin rpy="0 0 ${yaw}" xyz="-0.005 0 -0.002"/>
-    <limit effort="100" velocity="1.0" lower="${coxa_lower}" upper="${coxa_upper}"/>
+    <limit effort="100" velocity="2.0" lower="${coxa_lower}" upper="${coxa_upper}"/>
     <axis xyz="0 0 1"/>
     <!--dynamics damping="0.5" friction="0.0"/-->
@@ -124,5 +124,5 @@
     <child link="${name}_femur_link"/>
     <origin rpy="0 0 0" xyz="${servo_x} 0 0.005"/>
-    <limit effort="100" velocity="1.0" lower="-2.0" upper="0.7"/>
+    <limit effort="100" velocity="2.0" lower="-2.0" upper="0.7"/>
     <axis xyz="1 0 0"/>
     <!--dynamics damping="0.5" friction="0.0"/-->
@@ -165,5 +165,5 @@
     <child link="${name}_tibia_servo"/>
     <origin rpy="0 0 0" xyz="0 -0.055 0"/>
-    <limit effort="100" velocity="1.0" lower="-4.0" upper="1.0"/>
+    <limit effort="100" velocity="2.0" lower="-4.0" upper="1.0"/>
     <axis xyz="1 0 0"/>
     <!--dynamics damping="0.5" friction="0.0"/-->
@@ -231,9 +231,9 @@
   <!-- Rubber surface -->
   <gazebo reference="${name}_tibia_link">
-    <mu1 value="5.0"/>
-    <mu2 value="0.5"/>
-    <kp value="10000000.0" />
+    <mu1 value="1.0"/>
+    <mu2 value="1.0"/>
+    <kp value="100000.0" />
     <kd value="1.0" />
-    <fdir1 value="1 1 0"/>
+    <fdir1 value="0 1 0"/>
     <turnGravityOff>false</turnGravityOff>
     <selfCollide>true</selfCollide>

Commit message: "normalized" servo inputs

File: urdf/leg.xacro (robot description, xacro)
@@ -131,6 +131,6 @@
     <parent link="${name}_femur_servo"/>
     <child link="${name}_femur_link"/>
-    <origin rpy="0 0 0" xyz="${servo_x} 0 0.005"/>
-    <limit effort="${servo_effort}" velocity="${servo_velocity}" lower="-2.0" upper="0.7"/>
+    <origin rpy="${-pi/8} 0 0" xyz="${servo_x} 0 0.005"/>
+    <limit effort="${servo_effort}" velocity="${servo_velocity}" lower="-1.0" upper="1.0"/>
     <axis xyz="1 0 0"/>
   </joint>
@@ -175,6 +175,6 @@
     <parent link="${name}_femur_link"/>
     <child link="${name}_tibia_servo"/>
-    <origin rpy="0 0 0" xyz="0 -0.055 0"/>
-    <limit effort="${servo_effort}" velocity="${servo_velocity}" lower="-4.0" upper="1.0"/>
+    <origin rpy="${-pi/8} 0 0" xyz="0 -0.055 0"/>
+    <limit effort="${servo_effort}" velocity="${servo_velocity}" lower="-1.0" upper="1.0"/>
     <axis xyz="1 0 0"/>
     <dynamics friction="0.7"/>
@@ -245,5 +245,5 @@
     <kp value="10000000.0" />
     <kd value="1.0" />
-    <fdir1 value="1 0 0"/> <!-- sideways friction, hopefully -->
+    <fdir1 value="1 0 0"/>
     <turnGravityOff>false</turnGravityOff>
     <selfCollide>true</selfCollide>

Commit message: joint rotations in sync

File: urdf/leg.xacro (robot description, xacro)
@@ -133,5 +133,5 @@
     <origin rpy="${-pi/8} 0 0" xyz="${servo_x} 0 0.005"/>
     <limit effort="${servo_effort}" velocity="${servo_velocity}" lower="-1.0" upper="1.0"/>
-    <axis xyz="1 0 0"/>
+    <axis xyz="${-1*side} 0 0"/>
   </joint>
   <transmission name="${name}_femur_transmission">
@@ -177,5 +177,5 @@
     <origin rpy="${-pi/8} 0 0" xyz="0 -0.055 0"/>
     <limit effort="${servo_effort}" velocity="${servo_velocity}" lower="-1.0" upper="1.0"/>
-    <axis xyz="1 0 0"/>
+    <axis xyz="${side} 0 0"/>
     <dynamics friction="0.7"/>
   </joint>
