Commit message: visual urdf

File: urdf/critter.xacro (robot description, xacro)
@@ -11,6 +11,15 @@
     </visual>
   </link>
-  <xacro:leg name="front_left" parent_link="base_link">
+  <xacro:odd_leg name="front_left" parent_link="base_link">
     <origin xyz="0.03 0.035 0.0225" rpy="0 0 ${pi}"/>
-  </xacro:leg>
+  </xacro:odd_leg>
+  <xacro:even_leg name="rear_left" parent_link="base_link">
+    <origin xyz="-0.03 0.035 0.0225" rpy="0 0 0"/>
+  </xacro:even_leg>
+  <xacro:odd_leg name="rear_right" parent_link="base_link">
+    <origin xyz="-0.03 -0.035 0.0225" rpy="0 0 0"/>
+  </xacro:odd_leg>
+  <xacro:even_leg name="front_right" parent_link="base_link">
+    <origin xyz="0.03 -0.035 0.0225" rpy="0 0 ${pi}"/>
+  </xacro:even_leg>
 </robot>

File: urdf/leg.xacro (robot description, xacro)
@@ -1,5 +1,6 @@
 <?xml version="1.0"?>
 <robot xmlns:xacro="http://www.ros.org/wiki/xacro">
-  <xacro:macro name="leg" params="name parent_link *origin">
+  <!-- one kind of leg -->
+  <xacro:macro name="odd_leg" params="name parent_link *origin">
     <joint name="${name}_coxa_base_joint" type="fixed">
       <parent link="${parent_link}"/>
@@ -19,5 +20,5 @@
       <child link="${name}_coxa_link"/>
       <origin rpy="0 0 0" xyz="-0.005 0 -0.002"/>
-      <limit effort="100" velocity="0.1" lower="-2.0" upper="0.7"/>
+      <limit effort="100" velocity="0.1" lower="-1.7" upper="0.7"/>
       <axis xyz="0 0 1"/>
     </joint>
@@ -87,3 +88,90 @@
     </link>
 </xacro:macro>
+<!-- the other kind of leg -->
+<xacro:macro name="even_leg" params="name parent_link *origin">
+  <joint name="${name}_coxa_base_joint" type="fixed">
+    <parent link="${parent_link}"/>
+    <child link="${name}_coxa_servo"/>
+    <xacro:insert_block name="origin"/>
+  </joint>
+  <link name="${name}_coxa_servo">
+    <visual>
+      <origin rpy="0 0 0" xyz="0 0 0"/>
+      <geometry>
+        <mesh filename="package://open_critter/meshes/collada/servo.dae"/>
+      </geometry>
+    </visual>
+  </link>
+  <joint name="${name}_coxa_servo_joint" type="revolute">
+    <parent link="${name}_coxa_servo"/>
+    <child link="${name}_coxa_link"/>
+    <origin rpy="0 0 ${pi}" xyz="-0.005 0 -0.002"/>
+    <limit effort="100" velocity="0.1" lower="-0.7" upper="1.7"/>
+    <axis xyz="0 0 1"/>
+  </joint>
+  <link name="${name}_coxa_link">
+    <visual>
+    <origin rpy="0 0 ${pi}" xyz="-0.002 -0.016 0"/>
+      <geometry>
+        <mesh filename="package://open_critter/meshes/collada/coxa_rear.dae"/>
+      </geometry>
+    </visual>
+  </link>
+  <joint name="${name}_femur_servo_coxa_joint" type="fixed">
+    <parent link="${name}_coxa_link"/>
+    <child link="${name}_femur_servo"/>
+    <origin rpy="0 0 0" xyz="-0.005 -0.0275 0"/>
+  </joint>
+  <link name="${name}_femur_servo">
+    <visual>
+      <origin rpy="0 ${pi/2} ${pi}" xyz="0 0 0"/>
+      <geometry>
+        <mesh filename="package://open_critter/meshes/collada/servo.dae"/>
+      </geometry>
+    </visual>
+  </link>
+  <joint name="${name}_femur_servo_joint" type="revolute">
+    <parent link="${name}_femur_servo"/>
+    <child link="${name}_femur_link"/>
+    <origin rpy="0 0 0" xyz="0 0 0.005"/>
+    <limit effort="100" velocity="0.1" lower="-2.0" upper="0.7"/>
+    <axis xyz="1 0 0"/>
+  </joint>
+  <link name="${name}_femur_link">
+    <visual>
+    <origin rpy="0 ${pi} 0" xyz="0.0025 -0.0275 0"/>
+      <geometry>
+        <mesh filename="package://open_critter/meshes/collada/femur.dae"/>
+      </geometry>
+    </visual>
+  </link>
+  <joint name="${name}_tibia_servo_joint" type="revolute">
+    <parent link="${name}_femur_link"/>
+    <child link="${name}_tibia_servo"/>
+    <origin rpy="0 0 0" xyz="0 -0.055 0"/>
+    <limit effort="100" velocity="0.1" lower="-4.0" upper="1.0"/>
+    <axis xyz="1 0 0"/>
+  </joint>
+  <link name="${name}_tibia_servo">
+    <visual>
+      <origin rpy="0 ${pi/2} ${pi}" xyz="0 0 -0.005"/>
+      <geometry>
+        <mesh filename="package://open_critter/meshes/collada/servo.dae"/>
+      </geometry>
+    </visual>
+  </link>
+  <joint name="${name}_tibia_servo_femur_joint" type="fixed">
+    <parent link="${name}_tibia_servo"/>
+    <child link="${name}_tibia_link"/>
+    <origin rpy="0 0 0" xyz="0 0 0"/>
+  </joint>
+  <link name="${name}_tibia_link">
+    <visual>
+      <origin rpy="0 0 ${pi}" xyz="0.007 0 -0.03"/>
+      <geometry>
+        <mesh filename="package://open_critter/meshes/collada/tibia_front.dae"/>
+      </geometry>
+    </visual>
+  </link>
+</xacro:macro>
 </robot>

Commit message: leg macro refact

File: urdf/critter.xacro (robot description, xacro)
@@ -10,16 +10,22 @@
       </geometry>
     </visual>
+    <collision>
+      <origin rpy="0 0 3.14" xyz="0.0 0.0 0.04"/>
+      <geometry>
+        <mesh filename="package://open_critter/meshes/collada/body.dae"/>
+      </geometry>
+    </collision>
   </link>
-  <xacro:odd_leg name="front_left" parent_link="base_link">
+  <xacro:leg name="front_left" odd="true" parent_link="base_link">
     <origin xyz="0.03 0.035 0.0225" rpy="0 0 ${pi}"/>
-  </xacro:odd_leg>
-  <xacro:even_leg name="rear_left" parent_link="base_link">
+  </xacro:leg>
+  <xacro:leg name="rear_left" odd="false" parent_link="base_link">
     <origin xyz="-0.03 0.035 0.0225" rpy="0 0 0"/>
-  </xacro:even_leg>
-  <xacro:odd_leg name="rear_right" parent_link="base_link">
+  </xacro:leg>
+  <xacro:leg name="rear_right" odd="true" parent_link="base_link">
     <origin xyz="-0.03 -0.035 0.0225" rpy="0 0 0"/>
-  </xacro:odd_leg>
-  <xacro:even_leg name="front_right" parent_link="base_link">
+  </xacro:leg>
+  <xacro:leg name="front_right" odd="false" parent_link="base_link">
     <origin xyz="0.03 -0.035 0.0225" rpy="0 0 ${pi}"/>
-  </xacro:even_leg>
+  </xacro:leg>
 </robot>

File: urdf/leg.xacro (robot description, xacro)
@@ -1,126 +1,28 @@
 <?xml version="1.0"?>
 <robot xmlns:xacro="http://www.ros.org/wiki/xacro">
-  <!-- one kind of leg -->
-  <xacro:macro name="odd_leg" params="name parent_link *origin">
-    <joint name="${name}_coxa_base_joint" type="fixed">
-      <parent link="${parent_link}"/>
-      <child link="${name}_coxa_servo"/>
-      <xacro:insert_block name="origin"/>
-    </joint>
-    <link name="${name}_coxa_servo">
-      <visual>
-        <origin rpy="0 0 0" xyz="0 0 0"/>
-        <geometry>
-          <mesh filename="package://open_critter/meshes/collada/servo.dae"/>
-        </geometry>
-      </visual>
-    </link>
-    <joint name="${name}_coxa_servo_joint" type="revolute">
-      <parent link="${name}_coxa_servo"/>
-      <child link="${name}_coxa_link"/>
-      <origin rpy="0 0 0" xyz="-0.005 0 -0.002"/>
-      <limit effort="100" velocity="0.1" lower="-1.7" upper="0.7"/>
-      <axis xyz="0 0 1"/>
-    </joint>
-    <transmission name="${name}_coxa_servo_transmission">
-        <type>transmission_interface/SimpleTransmission</type>
-        <joint name="${name}_coxa_servo_joint">
-            <hardwareInterface>hardware_interface/PositionJointInterface</hardwareInterface>
-        </joint>
-        <actuator name="${name}_coxa_servo_actuator">
-            <hardwareInterface>hardware_interface/PositionJointInterface</hardwareInterface>
-            <mechanicalReduction>1</mechanicalReduction>
-            <motorTorqueConstant>1</motorTorqueConstant>
-        </actuator>
-    </transmission>
-    <link name="${name}_coxa_link">
-      <visual>
-      <origin rpy="0 0 0" xyz="0.002 -0.016 0"/>
-        <geometry>
-          <mesh filename="package://open_critter/meshes/collada/coxa_front.dae"/>
-        </geometry>
-      </visual>
-    </link>
-    <joint name="${name}_femur_servo_coxa_joint" type="fixed">
-      <parent link="${name}_coxa_link"/>
-      <child link="${name}_femur_servo"/>
-      <origin rpy="0 0 0" xyz="-0.005 -0.0275 0"/>
-    </joint>
-    <link name="${name}_femur_servo">
-      <visual>
-        <origin rpy="0 ${pi/2} ${pi}" xyz="0 0 0"/>
-        <geometry>
-          <mesh filename="package://open_critter/meshes/collada/servo.dae"/>
-        </geometry>
-      </visual>
-    </link>
-    <joint name="${name}_femur_servo_joint" type="revolute">
-      <parent link="${name}_femur_servo"/>
-      <child link="${name}_femur_link"/>
-      <origin rpy="0 0 0" xyz="0 0 0.005"/>
-      <limit effort="100" velocity="0.1" lower="-2.0" upper="0.7"/>
-      <axis xyz="1 0 0"/>
-    </joint>
-    <transmission name="${name}_femur_servo_transmission">
-        <type>transmission_interface/SimpleTransmission</type>
-        <joint name="${name}_femur_servo_joint">
-            <hardwareInterface>hardware_interface/PositionJointInterface</hardwareInterface>
-        </joint>
-        <actuator name="${name}_femur_servo_actuator">
-            <hardwareInterface>hardware_interface/PositionJointInterface</hardwareInterface>
-            <mechanicalReduction>1</mechanicalReduction>
-            <motorTorqueConstant>1</motorTorqueConstant>
-        </actuator>
-    </transmission>
-    <link name="${name}_femur_link">
-      <visual>
-      <origin rpy="0 ${pi} 0" xyz="0.0025 -0.0275 0"/>
-        <geometry>
-          <mesh filename="package://open_critter/meshes/collada/femur.dae"/>
-        </geometry>
-      </visual>
-    </link>
-    <joint name="${name}_tibia_servo_joint" type="revolute">
-      <parent link="${name}_femur_link"/>
-      <child link="${name}_tibia_servo"/>
-      <origin rpy="0 0 0" xyz="0 -0.055 0"/>
-      <limit effort="100" velocity="0.1" lower="-4.0" upper="1.0"/>
-      <axis xyz="1 0 0"/>
-    </joint>
-    <transmission name="${name}_tibia_servo_transmission">
-        <type>transmission_interface/SimpleTransmission</type>
-        <joint name="${name}_tibia_servo_joint">
-            <hardwareInterface>hardware_interface/PositionJointInterface</hardwareInterface>
-        </joint>
-        <actuator name="${name}_tibia_servo_actuator">
-            <hardwareInterface>hardware_interface/PositionJointInterface</hardwareInterface>
-            <mechanicalReduction>1</mechanicalReduction>
-            <motorTorqueConstant>1</motorTorqueConstant>
-        </actuator>
-    </transmission>
-    <link name="${name}_tibia_servo">
-      <visual>
-        <origin rpy="0 ${pi/2} ${pi}" xyz="0 0 -0.005"/>
-        <geometry>
-          <mesh filename="package://open_critter/meshes/collada/servo.dae"/>
-        </geometry>
-      </visual>
-    </link>
-    <joint name="${name}_tibia_servo_femur_joint" type="fixed">
-      <parent link="${name}_tibia_servo"/>
-      <child link="${name}_tibia_link"/>
-      <origin rpy="0 0 0" xyz="0 0 0"/>
-    </joint>
-    <link name="${name}_tibia_link">
-      <visual>
-        <origin rpy="0 0 ${pi}" xyz="0.007 0 -0.03"/>
-        <geometry>
-          <mesh filename="package://open_critter/meshes/collada/tibia_front.dae"/>
-        </geometry>
-      </visual>
-    </link>
-</xacro:macro>
-<!-- the other kind of leg -->
-<xacro:macro name="even_leg" params="name parent_link *origin">
+<!-- ultimate leg-->
+<xacro:macro name="leg" params="name odd parent_link *origin">
+  <xacro:if value="${odd}">
+    <xacro:property name="coxa_model"  value="package://open_critter/meshes/collada/coxa_front.dae"/>
+    <xacro:property name="tibia_model" value="package://open_critter/meshes/collada/tibia_rear.dae"/>
+    <xacro:property name="yaw" value="0"/>
+    <xacro:property name="nyaw" value="${pi}"/>
+    <xacro:property name="coxa_upper" value="0.7"/>
+    <xacro:property name="coxa_lower" value="-1.7"/>
+    <xacro:property name="side" value="1.0"/>
+    <xacro:property name="servo_x" value="0"/>
+    <xacro:property name="tibia_x" value="0.0075"/>
+  </xacro:if>
+  <xacro:unless value="${odd}"> <!-- EVEN -->
+    <xacro:property name="coxa_model" value="package://open_critter/meshes/collada/coxa_rear.dae"/>
+    <xacro:property name="tibia_model" value="package://open_critter/meshes/collada/tibia_front.dae"/>
+    <xacro:property name="yaw" value="${pi}"/>
+    <xacro:property name="nyaw" value="0"/>
+    <xacro:property name="coxa_upper" value="1.7"/>
+    <xacro:property name="coxa_lower" value="-0.7"/>
+    <xacro:property name="side" value="-1.0"/>
+    <xacro:property name="servo_x" value="-0.005"/>
+    <xacro:property name="tibia_x" value="-0.0025"/>
+  </xacro:unless>
   <joint name="${name}_coxa_base_joint" type="fixed">
     <parent link="${parent_link}"/>
@@ -139,6 +41,6 @@
     <parent link="${name}_coxa_servo"/>
     <child link="${name}_coxa_link"/>
-    <origin rpy="0 0 ${pi}" xyz="-0.005 0 -0.002"/>
-    <limit effort="100" velocity="0.1" lower="-0.7" upper="1.7"/>
+    <origin rpy="0 0 ${yaw}" xyz="-0.005 0 -0.002"/>
+    <limit effort="100" velocity="0.1" lower="${coxa_lower}" upper="${coxa_upper}"/>
     <axis xyz="0 0 1"/>
   </joint>
@@ -156,7 +58,7 @@
   <link name="${name}_coxa_link">
     <visual>
-    <origin rpy="0 0 ${pi}" xyz="-0.002 -0.016 0"/>
+    <origin rpy="0 0 ${yaw}" xyz="${side*0.002} -0.016 0"/>
       <geometry>
-        <mesh filename="package://open_critter/meshes/collada/coxa_rear.dae"/>
+        <mesh filename="${coxa_model}"/>
       </geometry>
     </visual>
@@ -165,9 +67,9 @@
     <parent link="${name}_coxa_link"/>
     <child link="${name}_femur_servo"/>
-    <origin rpy="0 0 0" xyz="-0.005 -0.0275 0"/>
+    <origin rpy="0 0 0" xyz="${side*-0.005} -0.0275 0"/>
   </joint>
   <link name="${name}_femur_servo">
     <visual>
-      <origin rpy="0 ${pi/2} ${pi}" xyz="0 0 0"/>
+      <origin rpy="0 ${pi/2} ${nyaw}" xyz="0 0 0"/>
       <geometry>
         <mesh filename="package://open_critter/meshes/collada/servo.dae"/>
@@ -178,5 +80,5 @@
     <parent link="${name}_femur_servo"/>
     <child link="${name}_femur_link"/>
-    <origin rpy="0 0 0" xyz="0 0 0.005"/>
+    <origin rpy="0 0 0" xyz="${servo_x} 0 0.005"/>
     <limit effort="100" velocity="0.1" lower="-2.0" upper="0.7"/>
     <axis xyz="1 0 0"/>
@@ -195,5 +97,5 @@
   <link name="${name}_femur_link">
     <visual>
-    <origin rpy="0 ${pi} 0" xyz="0.0025 -0.0275 0"/>
+    <origin rpy="0 ${nyaw} 0" xyz="0.0025 -0.0275 0"/>
       <geometry>
         <mesh filename="package://open_critter/meshes/collada/femur.dae"/>
@@ -221,5 +123,5 @@
   <link name="${name}_tibia_servo">
     <visual>
-      <origin rpy="0 ${pi/2} ${pi}" xyz="0 0 -0.005"/>
+      <origin rpy="0 ${pi/2} ${nyaw}" xyz="${side*servo_x} 0 -0.005"/>
       <geometry>
         <mesh filename="package://open_critter/meshes/collada/servo.dae"/>
@@ -234,7 +136,7 @@
   <link name="${name}_tibia_link">
     <visual>
-      <origin rpy="0 0 0" xyz="0.007 0 -0.03"/>
+      <origin rpy="0 0 ${nyaw}" xyz="${tibia_x} 0 -0.03"/>
       <geometry>
-        <mesh filename="package://open_critter/meshes/collada/tibia_rear.dae"/>
+        <mesh filename="${tibia_model}"/>
       </geometry>
     </visual>
