Commit message: joint position interfaces

File: urdf/critter.xacro (robot description, xacro)
@@ -16,4 +16,12 @@
       </geometry>
     </collision>
+    <inertial>
+      <origin rpy="0 0 0" xyz="0 0 0"/>
+      <geometry>
+        <box size="0.1 0.05 0.03"/>
+      </geometry>
+        <mass value="0.2"/>
+        <box_inertia m="0.2" x="0.1" y="0.05" z="0.03" />
+    </inertial>
   </link>
   <xacro:leg name="front_left" odd="true" parent_link="base_link">
@@ -29,3 +37,8 @@
     <origin xyz="0.03 -0.035 0.0225" rpy="0 0 ${pi}"/>
   </xacro:leg>
+  <gazebo>
+      <plugin name="gazebo_ros_control" filename="libgazebo_ros_control.so">
+          <robotNamespace>/open_critter</robotNamespace>
+      </plugin>
+  </gazebo>
 </robot>

File: urdf/leg.xacro (robot description, xacro)
@@ -25,5 +25,5 @@
     <xacro:property name="tibia_x" value="-0.0025"/>
   </xacro:unless>
-  <joint name="${name}_coxa_base_joint" type="fixed">
+  <joint name="${name}_base" type="fixed">
     <parent link="${parent_link}"/>
     <child link="${name}_coxa_servo"/>
@@ -37,21 +37,36 @@
       </geometry>
     </visual>
-  </link>
-  <joint name="${name}_coxa_servo_joint" type="revolute">
+    <collision>
+      <origin rpy="0 0 0" xyz="0 0 0"/>
+      <geometry>
+        <mesh filename="package://open_critter/meshes/collada/servo.dae"/>
+      </geometry>
+    </collision>
+    <inertial>
+      <origin rpy="0 0 0" xyz="0 0 0"/>
+      <geometry>
+        <box size="0.02 0.01 0.03"/>
+      </geometry>
+        <mass value="0.009"/>
+        <box_inertia m="0.009" x="0.02" y="0.01" z="0.03" />
+    </inertial>
+  </link>
+  <joint name="${name}_coxa_joint" type="revolute">
     <parent link="${name}_coxa_servo"/>
     <child link="${name}_coxa_link"/>
     <origin rpy="0 0 ${yaw}" xyz="-0.005 0 -0.002"/>
-    <limit effort="100" velocity="0.1" lower="${coxa_lower}" upper="${coxa_upper}"/>
+    <limit effort="100" velocity="1.0" lower="${coxa_lower}" upper="${coxa_upper}"/>
     <axis xyz="0 0 1"/>
-  </joint>
-  <transmission name="${name}_coxa_servo_transmission">
+    <!--dynamics damping="0.5" friction="0.0"/-->
+  </joint>
+  <transmission name="${name}_coxa_transmission">
       <type>transmission_interface/SimpleTransmission</type>
-      <joint name="${name}_coxa_servo_joint">
+      <joint name="${name}_coxa_joint">
           <hardwareInterface>hardware_interface/PositionJointInterface</hardwareInterface>
       </joint>
-      <actuator name="${name}_coxa_servo_actuator">
+      <actuator name="${name}_coxa_actuator">
           <hardwareInterface>hardware_interface/PositionJointInterface</hardwareInterface>
           <mechanicalReduction>1</mechanicalReduction>
-          <motorTorqueConstant>1</motorTorqueConstant>
+          <motorTorqueConstant>10</motorTorqueConstant>
       </actuator>
   </transmission>
@@ -63,6 +78,20 @@
       </geometry>
     </visual>
-  </link>
-  <joint name="${name}_femur_servo_coxa_joint" type="fixed">
+    <collision>
+    <origin rpy="0 0 ${yaw}" xyz="${side*0.002} -0.016 0"/>
+      <geometry>
+        <mesh filename="${coxa_model}"/>
+      </geometry>
+    </collision>
+    <inertial>
+      <origin rpy="0 0 0" xyz="0 0 0"/>
+      <geometry>
+        <box size="0.04 0.01 0.03"/>
+      </geometry>
+        <mass value="0.001"/>
+        <box_inertia m="0.001" x="0.04" y="0.01" z="0.03" />
+    </inertial>
+  </link>
+  <joint name="${name}_femur_servo_to_coxa_joint" type="fixed">
     <parent link="${name}_coxa_link"/>
     <child link="${name}_femur_servo"/>
@@ -76,21 +105,36 @@
       </geometry>
     </visual>
-  </link>
-  <joint name="${name}_femur_servo_joint" type="revolute">
+    <collision>
+      <origin rpy="0 ${pi/2} ${nyaw}" xyz="0 0 0"/>
+      <geometry>
+        <mesh filename="package://open_critter/meshes/collada/servo.dae"/>
+      </geometry>
+    </collision>
+    <inertial>
+      <origin rpy="0 ${pi/2} ${nyaw}" xyz="0 0 0"/>
+      <geometry>
+        <box size="0.02 0.01 0.03"/>
+      </geometry>
+        <mass value="0.009"/>
+        <box_inertia m="0.009" x="0.02" y="0.01" z="0.03" />
+    </inertial>
+  </link>
+  <joint name="${name}_femur_joint" type="revolute">
     <parent link="${name}_femur_servo"/>
     <child link="${name}_femur_link"/>
     <origin rpy="0 0 0" xyz="${servo_x} 0 0.005"/>
-    <limit effort="100" velocity="0.1" lower="-2.0" upper="0.7"/>
+    <limit effort="100" velocity="1.0" lower="-2.0" upper="0.7"/>
     <axis xyz="1 0 0"/>
-  </joint>
-  <transmission name="${name}_femur_servo_transmission">
+    <!--dynamics damping="0.5" friction="0.0"/-->
+  </joint>
+  <transmission name="${name}_femur_transmission">
       <type>transmission_interface/SimpleTransmission</type>
-      <joint name="${name}_femur_servo_joint">
+      <joint name="${name}_femur_joint">
           <hardwareInterface>hardware_interface/PositionJointInterface</hardwareInterface>
       </joint>
-      <actuator name="${name}_femur_servo_actuator">
+      <actuator name="${name}_femur_actuator">
           <hardwareInterface>hardware_interface/PositionJointInterface</hardwareInterface>
           <mechanicalReduction>1</mechanicalReduction>
-          <motorTorqueConstant>1</motorTorqueConstant>
+          <motorTorqueConstant>10</motorTorqueConstant>
       </actuator>
   </transmission>
@@ -102,21 +146,36 @@
       </geometry>
     </visual>
-  </link>
-  <joint name="${name}_tibia_servo_joint" type="revolute">
+    <collision>
+    <origin rpy="0 ${nyaw} 0" xyz="0.0025 -0.0275 0"/>
+      <geometry>
+        <mesh filename="package://open_critter/meshes/collada/femur.dae"/>
+      </geometry>
+    </collision>
+    <inertial>
+      <origin rpy="0 0 0" xyz="0 0 0"/>
+      <geometry>
+        <box size="0.05 0.01 0.03"/>
+      </geometry>
+        <mass value="0.002"/>
+        <box_inertia m="0.002" x="0.05" y="0.01" z="0.03" />
+    </inertial>
+  </link>
+  <joint name="${name}_tibia_joint" type="revolute">
     <parent link="${name}_femur_link"/>
     <child link="${name}_tibia_servo"/>
     <origin rpy="0 0 0" xyz="0 -0.055 0"/>
-    <limit effort="100" velocity="0.1" lower="-4.0" upper="1.0"/>
+    <limit effort="100" velocity="1.0" lower="-4.0" upper="1.0"/>
     <axis xyz="1 0 0"/>
-  </joint>
-  <transmission name="${name}_tibia_servo_transmission">
+    <!--dynamics damping="0.5" friction="0.0"/-->
+  </joint>
+  <transmission name="${name}_tibia_transmission">
       <type>transmission_interface/SimpleTransmission</type>
-      <joint name="${name}_tibia_servo_joint">
+      <joint name="${name}_tibia_joint">
           <hardwareInterface>hardware_interface/PositionJointInterface</hardwareInterface>
       </joint>
-      <actuator name="${name}_tibia_servo_actuator">
+      <actuator name="${name}_tibia_actuator">
           <hardwareInterface>hardware_interface/PositionJointInterface</hardwareInterface>
           <mechanicalReduction>1</mechanicalReduction>
-          <motorTorqueConstant>1</motorTorqueConstant>
+          <motorTorqueConstant>10</motorTorqueConstant>
       </actuator>
   </transmission>
@@ -128,6 +187,20 @@
       </geometry>
     </visual>
-  </link>
-  <joint name="${name}_tibia_servo_femur_joint" type="fixed">
+    <collision>
+      <origin rpy="0 ${pi/2} ${nyaw}" xyz="${side*servo_x} 0 -0.005"/>
+      <geometry>
+        <mesh filename="package://open_critter/meshes/collada/servo.dae"/>
+      </geometry>
+    </collision>
+    <inertial>
+      <origin rpy="0 ${pi/2} ${nyaw}" xyz="${side*servo_x} 0 -0.005"/>
+      <geometry>
+        <box size="0.02 0.01 0.03"/>
+      </geometry>
+        <mass value="0.009"/>
+        <box_inertia m="0.009" x="0.02" y="0.01" z="0.03" />
+    </inertial>
+  </link>
+  <joint name="${name}_tibia_servo_to_femur_joint" type="fixed">
     <parent link="${name}_tibia_servo"/>
     <child link="${name}_tibia_link"/>
@@ -141,5 +214,29 @@
       </geometry>
     </visual>
-  </link>
+    <collision>
+      <origin rpy="0 0 ${nyaw}" xyz="${tibia_x} 0 -0.03"/>
+      <geometry>
+        <mesh filename="${tibia_model}"/>
+      </geometry>
+    </collision>
+    <inertial>
+      <origin rpy="0 0 0" xyz="0 0 0"/>
+      <geometry>
+        <box size="0.1 0.005 0.005"/>
+      </geometry>
+        <mass value="0.001"/>
+        <box_inertia m="0.001" x="0.1" y="0.005" z="0.005" />
+    </inertial>
+  </link>
+  <!-- Rubber surface -->
+  <gazebo reference="${name}_tibia_link">
+    <mu1 value="5.0"/>
+    <mu2 value="0.5"/>
+    <kp value="10000000.0" />
+    <kd value="1.0" />
+    <fdir1 value="1 1 0"/>
+    <turnGravityOff>false</turnGravityOff>
+    <selfCollide>true</selfCollide>
+  </gazebo>
 </xacro:macro>
 </robot>

Commit message: controller init

File: urdf/critter.xacro (robot description, xacro)
@@ -3,4 +3,34 @@
   <xacro:include filename="$(find open_critter)/urdf/inertia.xacro"/>
   <xacro:include filename="$(find open_critter)/urdf/leg.xacro"/>
+  <xacro:property name="use_stand" value="false"/>
+  <xacro:if value="${use_stand}">
+    <link name="stand_link">
+      <visual>
+        <origin rpy="0 0 0" xyz="0 0 0"/>
+        <geometry>
+          <box size="0.2 0.2 0.02"/>
+        </geometry>
+      </visual>
+      <collision>
+        <origin rpy="0 0 0" xyz="0 0 0"/>
+        <geometry>
+          <box size="0.2 0.2 0.02"/>
+        </geometry>
+      </collision>
+      <inertial>
+        <origin rpy="0 0 0" xyz="0 0 0"/>
+        <geometry>
+          <box size="0.2 0.2 0.02"/>
+        </geometry>
+          <mass value="10.0"/>
+          <box_inertia m="10.0" x="0.2" y="0.2" z="0.02" />
+      </inertial>
+    </link>
+    <joint name="stand_joint" type="fixed">
+      <parent link="stand_link"/>
+      <child link="base_link"/>
+      <origin rpy="0 0 0" xyz="0.0 0.0 0.4"/>
+    </joint>
+  </xacro:if>
   <link name="base_link">
     <visual>

File: urdf/leg.xacro (robot description, xacro)
@@ -3,4 +3,8 @@
 <!-- ultimate leg-->
 <xacro:macro name="leg" params="name odd parent_link *origin">
+  <xacro:property name="servo_effort"    value="10"/>
+  <xacro:property name="servo_velocity"  value="10"/>
+  <xacro:property name="servo_torque"    value="2"/>
+  <xacro:property name="servo_reduction" value="1"/>
   <xacro:if value="${odd}">
     <xacro:property name="coxa_model"  value="package://open_critter/meshes/collada/coxa_front.dae"/>
@@ -56,7 +60,6 @@
     <child link="${name}_coxa_link"/>
     <origin rpy="0 0 ${yaw}" xyz="-0.005 0 -0.002"/>
-    <limit effort="100" velocity="2.0" lower="${coxa_lower}" upper="${coxa_upper}"/>
+    <limit effort="${servo_effort}" velocity="${servo_velocity}" lower="${coxa_lower}" upper="${coxa_upper}"/>
     <axis xyz="0 0 1"/>
-    <!--dynamics damping="0.5" friction="0.0"/-->
   </joint>
   <transmission name="${name}_coxa_transmission">
@@ -67,6 +70,6 @@
       <actuator name="${name}_coxa_actuator">
           <hardwareInterface>hardware_interface/PositionJointInterface</hardwareInterface>
-          <mechanicalReduction>1</mechanicalReduction>
-          <motorTorqueConstant>10</motorTorqueConstant>
+          <mechanicalReduction>${servo_reduction}</mechanicalReduction>
+          <motorTorqueConstant>${servo_torque}</motorTorqueConstant>
       </actuator>
   </transmission>
@@ -124,7 +127,6 @@
     <child link="${name}_femur_link"/>
     <origin rpy="0 0 0" xyz="${servo_x} 0 0.005"/>
-    <limit effort="100" velocity="2.0" lower="-2.0" upper="0.7"/>
+    <limit effort="${servo_effort}" velocity="${servo_velocity}" lower="-2.0" upper="0.7"/>
     <axis xyz="1 0 0"/>
-    <!--dynamics damping="0.5" friction="0.0"/-->
   </joint>
   <transmission name="${name}_femur_transmission">
@@ -135,6 +137,6 @@
       <actuator name="${name}_femur_actuator">
           <hardwareInterface>hardware_interface/PositionJointInterface</hardwareInterface>
-          <mechanicalReduction>1</mechanicalReduction>
-          <motorTorqueConstant>10</motorTorqueConstant>
+          <mechanicalReduction>${servo_reduction}</mechanicalReduction>
+          <motorTorqueConstant>${servo_torque}</motorTorqueConstant>
       </actuator>
   </transmission>
@@ -165,7 +167,6 @@
     <child link="${name}_tibia_servo"/>
     <origin rpy="0 0 0" xyz="0 -0.055 0"/>
-    <limit effort="100" velocity="2.0" lower="-4.0" upper="1.0"/>
+    <limit effort="${servo_effort}" velocity="${servo_velocity}" lower="-4.0" upper="1.0"/>
     <axis xyz="1 0 0"/>
-    <!--dynamics damping="0.5" friction="0.0"/-->
   </joint>
   <transmission name="${name}_tibia_transmission">
@@ -176,6 +177,6 @@
       <actuator name="${name}_tibia_actuator">
           <hardwareInterface>hardware_interface/PositionJointInterface</hardwareInterface>
-          <mechanicalReduction>1</mechanicalReduction>
-          <motorTorqueConstant>10</motorTorqueConstant>
+          <mechanicalReduction>${servo_reduction}</mechanicalReduction>
+          <motorTorqueConstant>${servo_torque}</motorTorqueConstant>
       </actuator>
   </transmission>
@@ -229,6 +230,5 @@
     </inertial>
   </link>
-  <!-- Rubber surface -->
-  <gazebo reference="${name}_tibia_link">
+  <!-- <gazebo reference="${name}_tibia_link">
     <mu1 value="1.0"/>
     <mu2 value="1.0"/>
@@ -238,5 +238,5 @@
     <turnGravityOff>false</turnGravityOff>
     <selfCollide>true</selfCollide>
-  </gazebo>
+  </gazebo> -->
 </xacro:macro>
 </robot>

Commit message: rubber paw
still sliding

File: urdf/critter.xacro (robot description, xacro)
@@ -55,14 +55,15 @@
     </inertial>
   </link>
-  <xacro:leg name="front_left" odd="true" parent_link="base_link">
+  <xacro:property name="rubber_paw" value="true"/>
+  <xacro:leg name="front_left" odd="true" paw="${rubber_paw}" parent_link="base_link">
     <origin xyz="0.03 0.035 0.0225" rpy="0 0 ${pi}"/>
   </xacro:leg>
-  <xacro:leg name="rear_left" odd="false" parent_link="base_link">
+  <xacro:leg name="rear_left" odd="false" paw="${rubber_paw}" parent_link="base_link">
     <origin xyz="-0.03 0.035 0.0225" rpy="0 0 0"/>
   </xacro:leg>
-  <xacro:leg name="rear_right" odd="true" parent_link="base_link">
+  <xacro:leg name="rear_right" odd="true" paw="${rubber_paw}" parent_link="base_link">
     <origin xyz="-0.03 -0.035 0.0225" rpy="0 0 0"/>
   </xacro:leg>
-  <xacro:leg name="front_right" odd="false" parent_link="base_link">
+  <xacro:leg name="front_right" odd="false" paw="${rubber_paw}" parent_link="base_link">
     <origin xyz="0.03 -0.035 0.0225" rpy="0 0 ${pi}"/>
   </xacro:leg>

File: urdf/leg.xacro (robot description, xacro)
@@ -2,8 +2,8 @@
 <robot xmlns:xacro="http://www.ros.org/wiki/xacro">
 <!-- ultimate leg-->
-<xacro:macro name="leg" params="name odd parent_link *origin">
-  <xacro:property name="servo_effort"    value="10"/>
-  <xacro:property name="servo_velocity"  value="10"/>
-  <xacro:property name="servo_torque"    value="2"/>
+<xacro:macro name="leg" params="name odd parent_link paw *origin">
+  <xacro:property name="servo_effort"    value="1"/>
+  <xacro:property name="servo_velocity"  value="5"/>
+  <xacro:property name="servo_torque"    value="1"/>
   <xacro:property name="servo_reduction" value="1"/>
   <xacro:if value="${odd}">
@@ -17,4 +17,5 @@
     <xacro:property name="servo_x" value="0"/>
     <xacro:property name="tibia_x" value="0.0075"/>
+    <xacro:property name="paw_x" value="0.0015"/>
   </xacro:if>
   <xacro:unless value="${odd}"> <!-- EVEN -->
@@ -28,4 +29,5 @@
     <xacro:property name="servo_x" value="-0.005"/>
     <xacro:property name="tibia_x" value="-0.0025"/>
+    <xacro:property name="paw_x" value="0.0035"/>
   </xacro:unless>
   <joint name="${name}_base" type="fixed">
@@ -169,4 +171,5 @@
     <limit effort="${servo_effort}" velocity="${servo_velocity}" lower="-4.0" upper="1.0"/>
     <axis xyz="1 0 0"/>
+    <dynamics friction="0.7"/>
   </joint>
   <transmission name="${name}_tibia_transmission">
@@ -230,13 +233,64 @@
     </inertial>
   </link>
-  <!-- <gazebo reference="${name}_tibia_link">
-    <mu1 value="1.0"/>
-    <mu2 value="1.0"/>
-    <kp value="100000.0" />
-    <kd value="1.0" />
-    <fdir1 value="0 1 0"/>
-    <turnGravityOff>false</turnGravityOff>
-    <selfCollide>true</selfCollide>
-  </gazebo> -->
+  <!-- RUBBER BALL PAW -->
+  <xacro:if value="${paw}">
+    <joint name="${name}_tibia_paw_joint" type="fixed">
+      <parent link="${name}_tibia_link"/>
+      <child link="${name}_paw_link"/>
+      <origin rpy="0 0 0" xyz="${paw_x} 0 -0.08"/>
+    </joint>
+    <link name="${name}_paw_link">
+      <visual>
+        <origin rpy="0 0 0" xyz="0 0 0"/>
+        <geometry>
+          <sphere radius="0.005"/>
+        </geometry>
+      </visual>
+      <collision>
+        <origin rpy="0 0 0" xyz="0 0 0"/>
+        <geometry>
+          <sphere radius="0.005"/>
+        </geometry>
+      </collision>
+      <inertial>
+        <origin rpy="0 0 0" xyz="0 0 0"/>
+        <geometry>
+          <sphere radius="0.005"/>
+        </geometry>
+          <mass value="0.001"/>
+          <sphere_inertia m="0.001" r="0.005"/>
+      </inertial>
+    </link>
+    <gazebo reference="${name}_paw_link">
+      <mu1>1</mu1>
+      <mu2>1</mu2>
+      <fdir1>1 0 0</fdir1>
+      <maxContacts>1</maxContacts>
+      <minDepth>0.005</minDepth>
+      <gravity>true</gravity>
+      <collision name="${name}__paw_link_collision">
+        <geometry>
+            <sphere>
+            <radius>0.005</radius>
+        </sphere>
+        </geometry>
+        <surface>
+          <friction>
+            <torsional>
+                <coefficient>10</coefficient>
+                <use_patch_radius>true</use_patch_radius>
+                <surface_radius>0.05</surface_radius>
+                <patch_radius>0.01</patch_radius>
+            </torsional>
+          </friction>
+          <contact>
+            <poissons_ratio>0.5</poissons_ratio>
+            <elastic_modulus>1e8</elastic_modulus>
+          </contact>
+        </surface>
+      </collision>
+      <material>Gazebo/Red</material>
+    </gazebo>
+  </xacro:if>
 </xacro:macro>
 </robot>

Commit message: simple servo test

File: urdf/critter.xacro (robot description, xacro)
@@ -55,5 +55,12 @@
     </inertial>
   </link>
-  <xacro:property name="rubber_paw" value="true"/>
+  <!-- <gazebo reference="base_link">
+    <selfCollide>True</selfCollide>
+    <mu1 value="200.0"/>
+    <mu2 value="100.0"/>
+    <kp value="10000000.0"/>
+    <kd value="1.0"/>
+  </gazebo> -->
+  <xacro:property name="rubber_paw" value="false"/>
   <xacro:leg name="front_left" odd="true" paw="${rubber_paw}" parent_link="base_link">
     <origin xyz="0.03 0.035 0.0225" rpy="0 0 ${pi}"/>
@@ -68,8 +75,8 @@
     <origin xyz="0.03 -0.035 0.0225" rpy="0 0 ${pi}"/>
   </xacro:leg>
-  <gazebo>
+  <!-- <gazebo>
       <plugin name="gazebo_ros_control" filename="libgazebo_ros_control.so">
           <robotNamespace>/open_critter</robotNamespace>
       </plugin>
-  </gazebo>
+  </gazebo> -->
 </robot>

File: urdf/leg.xacro (robot description, xacro)
@@ -1,6 +1,6 @@
 <?xml version="1.0"?>
 <robot xmlns:xacro="http://www.ros.org/wiki/xacro">
-<!-- ultimate leg-->
 <xacro:macro name="leg" params="name odd parent_link paw *origin">
+  <xacro:property name="servo_ns"        value="open_critter"/>
   <xacro:property name="servo_effort"    value="1"/>
   <xacro:property name="servo_velocity"  value="5"/>
@@ -65,5 +65,6 @@
     <axis xyz="0 0 1"/>
   </joint>
-  <transmission name="${name}_coxa_transmission">
+  <!--
+ <transmission name="${name}_coxa_transmission">
       <type>transmission_interface/SimpleTransmission</type>
       <joint name="${name}_coxa_joint">
@@ -75,5 +76,14 @@
           <motorTorqueConstant>${servo_torque}</motorTorqueConstant>
       </actuator>
-  </transmission>
+  </transmission> -->
+  <gazebo>
+    <plugin name="${name}_coxa" filename="libnowtech_gazebo_ros_simple_servo.so">
+       <update_rate>100.0</update_rate>
+       <actuator_velocity>0.1</actuator_velocity>
+       <actuated_joint>${name}_coxa_joint</actuated_joint>
+       <servo_name>${name}_coxa</servo_name>
+       <command_topic>${servo_ns}/${name}_coxa/command</command_topic>
+     </plugin>
+  </gazebo>
   <link name="${name}_coxa_link">
     <visual>
@@ -132,4 +142,5 @@
     <axis xyz="1 0 0"/>
   </joint>
+  <!--
   <transmission name="${name}_femur_transmission">
       <type>transmission_interface/SimpleTransmission</type>
@@ -142,5 +153,14 @@
           <motorTorqueConstant>${servo_torque}</motorTorqueConstant>
       </actuator>
-  </transmission>
+  </transmission> -->
+  <gazebo>
+    <plugin name="${name}_femur" filename="libnowtech_gazebo_ros_simple_servo.so">
+       <update_rate>100.0</update_rate>
+       <actuator_velocity>0.1</actuator_velocity>
+       <actuated_joint>${name}_femur_joint</actuated_joint>
+       <servo_name>${name}_femur</servo_name>
+       <command_topic>${servo_ns}/${name}_femur/command</command_topic>
+     </plugin>
+  </gazebo>
   <link name="${name}_femur_link">
     <visual>
@@ -173,4 +193,5 @@
     <dynamics friction="0.7"/>
   </joint>
+  <!--
   <transmission name="${name}_tibia_transmission">
       <type>transmission_interface/SimpleTransmission</type>
@@ -183,5 +204,14 @@
           <motorTorqueConstant>${servo_torque}</motorTorqueConstant>
       </actuator>
-  </transmission>
+  </transmission> -->
+  <gazebo>
+    <plugin name="${name}_tibia" filename="libnowtech_gazebo_ros_simple_servo.so">
+       <update_rate>100.0</update_rate>
+       <actuator_velocity>0.1</actuator_velocity>
+       <actuated_joint>${name}_tibia_joint</actuated_joint>
+       <servo_name>${name}_tibia</servo_name>
+       <command_topic>${servo_ns}/${name}_tibia/command</command_topic>
+     </plugin>
+  </gazebo>
   <link name="${name}_tibia_servo">
     <visual>
@@ -233,4 +263,12 @@
     </inertial>
   </link>
+  <gazebo reference="${name}_tibia_link">
+    <selfCollide>true</selfCollide>
+    <gravity>false</gravity>
+    <mu1 value="200.0"/>
+    <mu2 value="100.0"/>
+    <kp value="10000000.0"/>
+    <kd value="1.0"/>
+  </gazebo>
   <!-- RUBBER BALL PAW -->
   <xacro:if value="${paw}">
@@ -263,14 +301,17 @@
     </link>
     <gazebo reference="${name}_paw_link">
-      <mu1>1</mu1>
-      <mu2>1</mu2>
+      <mu1>0.6</mu1>
+      <mu2>0.85</mu2>
+      <kp>1000000.0</kp>
+      <kd>1.0</kd>
       <fdir1>1 0 0</fdir1>
       <maxContacts>1</maxContacts>
-      <minDepth>0.005</minDepth>
+      <minDepth>0.01</minDepth>
       <gravity>true</gravity>
+      <selfCollide>true</selfCollide>
       <collision name="${name}__paw_link_collision">
         <geometry>
             <sphere>
-            <radius>0.005</radius>
+            <radius>0.0055</radius>
         </sphere>
         </geometry>
