Commit message: doc update

File: urdf/critter.xacro (robot description, xacro)
@@ -4,4 +4,5 @@
   <xacro:include filename="$(find open_critter)/urdf/leg.xacro"/>
   <xacro:property name="use_stand" value="false"/>
+  <xacro:property name="rubber_paw" value="true"/>
   <xacro:if value="${use_stand}">
     <link name="stand_link">
@@ -55,5 +56,4 @@
     </inertial>
   </link>
-  <xacro:property name="rubber_paw" value="true"/>
   <xacro:leg name="front_left" odd="true" paw="${rubber_paw}" parent_link="base_link">
     <origin xyz="0.03 0.035 0.0225" rpy="0 0 ${pi}"/>

File: urdf/leg.xacro (robot description, xacro)
@@ -1,10 +1,9 @@
 <?xml version="1.0"?>
 <robot xmlns:xacro="http://www.ros.org/wiki/xacro">
-<!-- ultimate leg-->
 <xacro:macro name="leg" params="name odd parent_link paw *origin">
-  <xacro:property name="servo_effort"    value="1"/>
-  <xacro:property name="servo_velocity"  value="5"/>
-  <xacro:property name="servo_torque"    value="1"/>
-  <xacro:property name="servo_reduction" value="1"/>
+  <xacro:property name="servo_effort"    value="10"/>
+  <xacro:property name="servo_velocity"  value="4.0"/>
+  <xacro:property name="servo_torque"    value="10"/>
+  <xacro:property name="servo_reduction" value="1.0"/>
   <xacro:if value="${odd}">
     <xacro:property name="coxa_model"  value="package://open_critter/meshes/collada/coxa_front.dae"/>
@@ -43,10 +42,10 @@
       </geometry>
     </visual>
-    <collision>
-      <origin rpy="0 0 0" xyz="0 0 0"/>
-      <geometry>
-        <mesh filename="package://open_critter/meshes/collada/servo.dae"/>
-      </geometry>
-    </collision>
+    <!-- <collision>
+      <origin rpy="0 0 0" xyz="0 0 0"/>
+      <geometry>
+        <mesh filename="package://open_critter/meshes/collada/servo.dae"/>
+      </geometry>
+    </collision> -->
     <inertial>
       <origin rpy="0 0 0" xyz="0 0 0"/>
@@ -98,4 +97,8 @@
     </inertial>
   </link>
+  <gazebo reference="${name}_coxa_link">
+    <gravity>true</gravity>
+    <selfCollide>true</selfCollide>
+  </gazebo>
   <joint name="${name}_femur_servo_to_coxa_joint" type="fixed">
     <parent link="${name}_coxa_link"/>
@@ -110,10 +113,10 @@
       </geometry>
     </visual>
-    <collision>
+    <!-- <collision>
       <origin rpy="0 ${pi/2} ${nyaw}" xyz="0 0 0"/>
       <geometry>
         <mesh filename="package://open_critter/meshes/collada/servo.dae"/>
       </geometry>
-    </collision>
+    </collision> -->
     <inertial>
       <origin rpy="0 ${pi/2} ${nyaw}" xyz="0 0 0"/>
@@ -165,4 +168,8 @@
     </inertial>
   </link>
+  <gazebo reference="${name}_femur_link">
+    <gravity>true</gravity>
+    <selfCollide>true</selfCollide>
+  </gazebo>
   <joint name="${name}_tibia_joint" type="revolute">
     <parent link="${name}_femur_link"/>
@@ -191,10 +198,10 @@
       </geometry>
     </visual>
-    <collision>
+    <!-- <collision>
       <origin rpy="0 ${pi/2} ${nyaw}" xyz="${side*servo_x} 0 -0.005"/>
       <geometry>
         <mesh filename="package://open_critter/meshes/collada/servo.dae"/>
       </geometry>
-    </collision>
+    </collision> -->
     <inertial>
       <origin rpy="0 ${pi/2} ${nyaw}" xyz="${side*servo_x} 0 -0.005"/>
@@ -233,4 +240,13 @@
     </inertial>
   </link>
+  <gazebo reference="${name}_tibia_link">
+    <mu1 value="5.0"/>
+    <mu2 value="0.5"/>
+    <kp value="10000000.0" />
+    <kd value="1.0" />
+    <fdir1 value="1 0 0"/> <!-- sideways friction, hopefully -->
+    <turnGravityOff>false</turnGravityOff>
+    <selfCollide>true</selfCollide>
+  </gazebo>
   <!-- RUBBER BALL PAW -->
   <xacro:if value="${paw}">
@@ -263,10 +279,13 @@
     </link>
     <gazebo reference="${name}_paw_link">
-      <mu1>1</mu1>
-      <mu2>1</mu2>
-      <fdir1>1 0 0</fdir1>
+      <gravity>true</gravity>
+      <selfCollide>true</selfCollide>
+      <mu1>5.0</mu1>
+      <mu2>0.5</mu2>
+      <kp>10000000.0</kp>
+      <kd>1.0</kd>
+      <fdir1>0 1 0</fdir1>
       <maxContacts>1</maxContacts>
-      <minDepth>0.005</minDepth>
-      <gravity>true</gravity>
+      <minDepth>0.001</minDepth>
       <collision name="${name}__paw_link_collision">
         <geometry>
@@ -279,11 +298,11 @@
             <torsional>
                 <coefficient>10</coefficient>
-                <use_patch_radius>true</use_patch_radius>
-                <surface_radius>0.05</surface_radius>
+                <use_patch_radius>false</use_patch_radius>
+                <surface_radius>0.01</surface_radius>
                 <patch_radius>0.01</patch_radius>
             </torsional>
           </friction>
           <contact>
-            <poissons_ratio>0.5</poissons_ratio>
+            <poissons_ratio>0.01</poissons_ratio>
             <elastic_modulus>1e8</elastic_modulus>
           </contact>

Commit message: changed to world solver

File: urdf/critter.xacro (robot description, xacro)
@@ -73,3 +73,15 @@
       </plugin>
   </gazebo>
+  <gazebo>
+      <plugin name="p3d_base_controller" filename="libgazebo_ros_p3d.so">
+          <alwaysOn>true</alwaysOn>
+          <updateRate>100.0</updateRate>
+          <bodyName>base_link</bodyName>
+          <topicName>/gazebo/odom</topicName>
+          <gaussianNoise>0.00001</gaussianNoise>
+          <frameName>world</frameName>
+          <xyzOffsets>0 0 0</xyzOffsets>
+          <rpyOffsets>0 0 0</rpyOffsets>
+      </plugin>
+  </gazebo>
 </robot>

File: urdf/leg.xacro (robot description, xacro)
@@ -6,11 +6,12 @@
   <xacro:property name="servo_torque"    value="10"/>
   <xacro:property name="servo_reduction" value="1.0"/>
+  <xacro:property name="coxa_lower" value="-1.0"/>
+  <xacro:property name="coxa_upper" value="1.0"/>
   <xacro:if value="${odd}">
     <xacro:property name="coxa_model"  value="package://open_critter/meshes/collada/coxa_front.dae"/>
     <xacro:property name="tibia_model" value="package://open_critter/meshes/collada/tibia_rear.dae"/>
     <xacro:property name="yaw" value="0"/>
+    <xacro:property name="cyaw" value="${-pi/4}"/>
     <xacro:property name="nyaw" value="${pi}"/>
-    <xacro:property name="coxa_upper" value="0.7"/>
-    <xacro:property name="coxa_lower" value="-1.7"/>
     <xacro:property name="side" value="1.0"/>
     <xacro:property name="servo_x" value="0"/>
@@ -22,7 +23,6 @@
     <xacro:property name="tibia_model" value="package://open_critter/meshes/collada/tibia_front.dae"/>
     <xacro:property name="yaw" value="${pi}"/>
+    <xacro:property name="cyaw" value="${pi+pi/4}"/>
     <xacro:property name="nyaw" value="0"/>
-    <xacro:property name="coxa_upper" value="1.7"/>
-    <xacro:property name="coxa_lower" value="-0.7"/>
     <xacro:property name="side" value="-1.0"/>
     <xacro:property name="servo_x" value="-0.005"/>
@@ -60,5 +60,5 @@
     <parent link="${name}_coxa_servo"/>
     <child link="${name}_coxa_link"/>
-    <origin rpy="0 0 ${yaw}" xyz="-0.005 0 -0.002"/>
+    <origin rpy="0 0 ${cyaw}" xyz="-0.005 0 -0.002"/>
     <limit effort="${servo_effort}" velocity="${servo_velocity}" lower="${coxa_lower}" upper="${coxa_upper}"/>
     <axis xyz="0 0 1"/>
@@ -281,11 +281,11 @@
       <gravity>true</gravity>
       <selfCollide>true</selfCollide>
-      <mu1>5.0</mu1>
-      <mu2>0.5</mu2>
-      <kp>10000000.0</kp>
+      <mu1>0.1</mu1>
+      <mu2>0.1</mu2>
+      <kp>1000000.0</kp>
       <kd>1.0</kd>
       <fdir1>0 1 0</fdir1>
       <maxContacts>1</maxContacts>
-      <minDepth>0.001</minDepth>
+      <minDepth>0.0001</minDepth>
       <collision name="${name}__paw_link_collision">
         <geometry>

Commit message: xacro namespace prefix

File: urdf/critter.xacro (robot description, xacro)
@@ -25,5 +25,5 @@
         </geometry>
           <mass value="10.0"/>
-          <box_inertia m="10.0" x="0.2" y="0.2" z="0.02" />
+          <xacro:box_inertia m="10.0" x="0.2" y="0.2" z="0.02" />
       </inertial>
     </link>
@@ -34,4 +34,10 @@
     </joint>
   </xacro:if>
+  <link name="base_footprint"/>
+  <joint name="stand_joint" type="fixed">
+    <parent link="base_footprint"/>
+    <child link="base_link"/>
+    <origin rpy="0 0 0" xyz="0.0 0.0 0.0"/>
+  </joint>
   <link name="base_link">
     <visual>
@@ -53,5 +59,5 @@
       </geometry>
         <mass value="0.2"/>
-        <box_inertia m="0.2" x="0.1" y="0.05" z="0.03" />
+        <xacro:box_inertia m="0.2" x="0.1" y="0.05" z="0.03" />
     </inertial>
   </link>

File: urdf/leg.xacro (robot description, xacro)
@@ -54,5 +54,5 @@
       </geometry>
         <mass value="0.009"/>
-        <box_inertia m="0.009" x="0.02" y="0.01" z="0.03" />
+        <xacro:box_inertia m="0.009" x="0.02" y="0.01" z="0.03" />
     </inertial>
   </link>
@@ -94,5 +94,5 @@
       </geometry>
         <mass value="0.001"/>
-        <box_inertia m="0.001" x="0.04" y="0.01" z="0.03" />
+        <xacro:box_inertia m="0.001" x="0.04" y="0.01" z="0.03" />
     </inertial>
   </link>
@@ -125,5 +125,5 @@
       </geometry>
         <mass value="0.009"/>
-        <box_inertia m="0.009" x="0.02" y="0.01" z="0.03" />
+        <xacro:box_inertia m="0.009" x="0.02" y="0.01" z="0.03" />
     </inertial>
   </link>
@@ -165,5 +165,5 @@
       </geometry>
         <mass value="0.002"/>
-        <box_inertia m="0.002" x="0.05" y="0.01" z="0.03" />
+        <xacro:box_inertia m="0.002" x="0.05" y="0.01" z="0.03" />
     </inertial>
   </link>
@@ -210,5 +210,5 @@
       </geometry>
         <mass value="0.009"/>
-        <box_inertia m="0.009" x="0.02" y="0.01" z="0.03" />
+        <xacro:box_inertia m="0.009" x="0.02" y="0.01" z="0.03" />
     </inertial>
   </link>
@@ -237,5 +237,5 @@
       </geometry>
         <mass value="0.001"/>
-        <box_inertia m="0.001" x="0.1" y="0.005" z="0.005" />
+        <xacro:box_inertia m="0.001" x="0.1" y="0.005" z="0.005" />
     </inertial>
   </link>
@@ -275,5 +275,5 @@
         </geometry>
           <mass value="0.001"/>
-          <sphere_inertia m="0.001" r="0.005"/>
+          <xacro:sphere_inertia m="0.001" r="0.005"/>
       </inertial>
     </link>
