Commit message: minimal pybullet-gym

File: xacro/critter.xacro (robot description, xacro)
@@ -1,8 +1,8 @@
 <?xml version="1.0"?>
 <robot name="open_critter" xmlns:xacro="http://www.ros.org/wiki/xacro">
-  <xacro:include filename="$(find open_critter)/urdf/inertia.xacro"/>
-  <xacro:include filename="$(find open_critter)/urdf/leg.xacro"/>
+  <xacro:include filename="$(find open_critter)/xacro/inertia.xacro"/>
+  <xacro:include filename="$(find open_critter)/xacro/leg.xacro"/>
   <xacro:property name="use_stand" value="false"/>
-  <xacro:property name="rubber_paw" value="true"/>
+  <xacro:property name="rubber_paw" value="false"/>
   <xacro:if value="${use_stand}">
     <link name="stand_link">

File: xacro/leg.xacro (robot description, xacro)
@@ -1,9 +1,10 @@
 <?xml version="1.0"?>
 <robot xmlns:xacro="http://www.ros.org/wiki/xacro">
+<xacro:include filename="$(find open_critter)/xacro/inertia.xacro"/>
 <xacro:macro name="leg" params="name odd parent_link paw *origin">
-  <xacro:property name="servo_effort"    value="10"/>
-  <xacro:property name="servo_velocity"  value="4.0"/>
-  <xacro:property name="servo_torque"    value="10"/>
-  <xacro:property name="servo_reduction" value="1.0"/>
+  <xacro:property name="servo_effort"    value="1.0"/>
+  <xacro:property name="servo_velocity"  value="1.0"/>
+  <xacro:property name="servo_torque"    value="0.5"/>
+  <xacro:property name="servo_reduction" value="10.0"/>
   <xacro:property name="coxa_lower" value="-1.0"/>
   <xacro:property name="coxa_upper" value="1.0"/>
@@ -281,6 +282,6 @@
       <gravity>true</gravity>
       <selfCollide>true</selfCollide>
-      <mu1>0.1</mu1>
-      <mu2>0.1</mu2>
+      <mu1>100.0</mu1>
+      <mu2>50.0</mu2>
       <kp>1000000.0</kp>
       <kd>1.0</kd>

Commit message: minor tweaks and doc

File: xacro/critter.xacro (robot description, xacro)
@@ -4,5 +4,5 @@
   <xacro:include filename="$(find open_critter)/xacro/leg.xacro"/>
   <xacro:property name="use_stand" value="false"/>
-  <xacro:property name="rubber_paw" value="false"/>
+  <xacro:property name="rubber_paw" value="true"/>
   <xacro:if value="${use_stand}">
     <link name="stand_link">

File: xacro/leg.xacro (robot description, xacro)
@@ -4,5 +4,5 @@
 <xacro:macro name="leg" params="name odd parent_link paw *origin">
   <xacro:property name="servo_effort"    value="1.0"/>
-  <xacro:property name="servo_velocity"  value="1.0"/>
+  <xacro:property name="servo_velocity"  value="4.0"/>
   <xacro:property name="servo_torque"    value="0.5"/>
   <xacro:property name="servo_reduction" value="10.0"/>
@@ -286,5 +286,5 @@
       <kp>1000000.0</kp>
       <kd>1.0</kd>
-      <fdir1>0 1 0</fdir1>
+      <fdir1>1 0 0</fdir1>
       <maxContacts>1</maxContacts>
       <minDepth>0.0001</minDepth>
@@ -299,7 +299,7 @@
             <torsional>
                 <coefficient>10</coefficient>
-                <use_patch_radius>false</use_patch_radius>
-                <surface_radius>0.01</surface_radius>
-                <patch_radius>0.01</patch_radius>
+                <use_patch_radius>true</use_patch_radius>
+                <surface_radius>0.1</surface_radius>
+                <patch_radius>0.1</patch_radius>
             </torsional>
           </friction>

Commit message: trajectory control and ddpg tf

File: xacro/critter.xacro (robot description, xacro)
@@ -74,4 +74,63 @@
     <origin xyz="0.03 -0.035 0.0225" rpy="0 0 ${pi}"/>
   </xacro:leg>
+  <xacro:property name="imu_size" value="0.01"/>
+  <xacro:property name="imu_mass" value="0.01"/>
+  <link name="imu_link">
+    <visual>
+      <geometry>
+        <box size="${imu_size} ${imu_size} ${imu_size}"/>
+      </geometry>
+      <material name="white"/>
+    </visual>
+    <collision>
+      <geometry>
+        <box size="${imu_size} ${imu_size} ${imu_size}"/>
+      </geometry>
+    </collision>
+    <xacro:box_inertia m="${imu_mass}" x="${imu_size}" y="${imu_size}" z="${imu_size}"/>
+  </link>
+  <joint name="base_imu_joint" type="fixed">
+    <parent link="base_link"/>
+    <child link="imu_link"/>
+    <origin xyz="0 0 0.02" rpy="0 0 0"/>
+  </joint>
+  <gazebo reference="imu_link">
+      <gravity>true</gravity>
+      <sensor name="imu_sensor" type="imu">
+          <always_on>true</always_on>
+          <update_rate>100</update_rate>
+          <visualize>false</visualize>
+          <plugin filename="libgazebo_ros_imu_sensor.so" name="imu_plugin">
+              <topicName>/open_critter/imu</topicName>
+              <bodyName>imu_link</bodyName>
+              <updateRateHZ>100.0</updateRateHZ>
+              <gaussianNoise>0.0001</gaussianNoise>
+              <xyzOffset>0 0 0</xyzOffset>
+              <rpyOffset>0 0 0</rpyOffset>
+              <frameName>imu_link</frameName>
+          </plugin>
+      </sensor>
+  </gazebo>
+  <gazebo>
+    <plugin name="joint_state_publisher" filename="libgazebo_ros_joint_state_publisher.so">
+      <robotNamespace>/open_critter</robotNamespace>
+      <jointName>
+        front_left_coxa_joint,
+        front_right_coxa_joint,
+        rear_right_coxa_joint,
+        rear_left_coxa_joint,
+        front_left_femur_joint,
+        front_right_femur_joint,
+        rear_right_femur_joint,
+        rear_left_femur_joint,
+        front_left_tibia_joint,
+        front_right_tibia_joint,
+        rear_right_tibia_joint,
+        rear_left_tibia_joint
+      </jointName>
+      <updateRate>60.0</updateRate>
+      <alwaysOn>true</alwaysOn>
+    </plugin>
+  </gazebo>
   <gazebo>
       <plugin name="gazebo_ros_control" filename="libgazebo_ros_control.so">

File: xacro/leg.xacro (robot description, xacro)
@@ -68,8 +68,10 @@
       <type>transmission_interface/SimpleTransmission</type>
       <joint name="${name}_coxa_joint">
-          <hardwareInterface>hardware_interface/PositionJointInterface</hardwareInterface>
+          <!-- <hardwareInterface>hardware_interface/PositionJointInterface</hardwareInterface> -->
+          <hardwareInterface>hardware_interface/EffortJointInterface</hardwareInterface>
       </joint>
       <actuator name="${name}_coxa_actuator">
-          <hardwareInterface>hardware_interface/PositionJointInterface</hardwareInterface>
+          <hardwareInterface>hardware_interface/EffortJointInterface</hardwareInterface>
+          <!-- <hardwareInterface>hardware_interface/PositionJointInterface</hardwareInterface> -->
           <mechanicalReduction>${servo_reduction}</mechanicalReduction>
           <motorTorqueConstant>${servo_torque}</motorTorqueConstant>
@@ -139,8 +141,10 @@
       <type>transmission_interface/SimpleTransmission</type>
       <joint name="${name}_femur_joint">
-          <hardwareInterface>hardware_interface/PositionJointInterface</hardwareInterface>
+          <!-- <hardwareInterface>hardware_interface/PositionJointInterface</hardwareInterface> -->
+          <hardwareInterface>hardware_interface/EffortJointInterface</hardwareInterface>
       </joint>
       <actuator name="${name}_femur_actuator">
-          <hardwareInterface>hardware_interface/PositionJointInterface</hardwareInterface>
+          <!-- <hardwareInterface>hardware_interface/PositionJointInterface</hardwareInterface> -->
+          <hardwareInterface>hardware_interface/EffortJointInterface</hardwareInterface>
           <mechanicalReduction>${servo_reduction}</mechanicalReduction>
           <motorTorqueConstant>${servo_torque}</motorTorqueConstant>
@@ -184,8 +188,10 @@
       <type>transmission_interface/SimpleTransmission</type>
       <joint name="${name}_tibia_joint">
-          <hardwareInterface>hardware_interface/PositionJointInterface</hardwareInterface>
+          <!-- <hardwareInterface>hardware_interface/PositionJointInterface</hardwareInterface> -->
+          <hardwareInterface>hardware_interface/EffortJointInterface</hardwareInterface>
       </joint>
       <actuator name="${name}_tibia_actuator">
-          <hardwareInterface>hardware_interface/PositionJointInterface</hardwareInterface>
+          <!-- <hardwareInterface>hardware_interface/PositionJointInterface</hardwareInterface> -->
+          <hardwareInterface>hardware_interface/EffortJointInterface</hardwareInterface>
           <mechanicalReduction>${servo_reduction}</mechanicalReduction>
           <motorTorqueConstant>${servo_torque}</motorTorqueConstant>
@@ -280,5 +286,5 @@
     </link>
     <gazebo reference="${name}_paw_link">
-      <gravity>true</gravity>
+      <!-- <gravity>true</gravity>
       <selfCollide>true</selfCollide>
       <mu1>100.0</mu1>
@@ -287,6 +293,6 @@
       <kd>1.0</kd>
       <fdir1>1 0 0</fdir1>
-      <maxContacts>1</maxContacts>
-      <minDepth>0.0001</minDepth>
+      <maxContacts>1</maxContacts> -->
+      <minDepth>0.0002</minDepth>
       <collision name="${name}__paw_link_collision">
         <geometry>
@@ -296,4 +302,18 @@
         </geometry>
         <surface>
+          <friction>
+            <ode>
+              <mu>100000.0</mu>
+              <mu2>100000.0</mu2>
+            </ode>
+            <torsional>
+              <coefficient>1000000</coefficient>
+              <use_patch_radius>true</use_patch_radius>
+              <surface_radius>0.005</surface_radius>
+              <patch_radius>0.005</patch_radius>
+            </torsional>
+          </friction>
+        </surface>
+        <!-- <surface>
           <friction>
             <torsional>
@@ -308,5 +328,5 @@
             <elastic_modulus>1e8</elastic_modulus>
           </contact>
-        </surface>
+        </surface> -->
       </collision>
       <material>Gazebo/Red</material>

Commit message: environment setup

File: xacro/critter.xacro (robot description, xacro)
@@ -58,6 +58,6 @@
         <box size="0.1 0.05 0.03"/>
       </geometry>
-        <mass value="0.2"/>
-        <xacro:box_inertia m="0.2" x="0.1" y="0.05" z="0.03" />
+        <mass value="1.0"/>
+        <xacro:box_inertia m="1.0" x="0.1" y="0.05" z="0.03" />
     </inertial>
   </link>

File: xacro/leg.xacro (robot description, xacro)
@@ -5,6 +5,6 @@
   <xacro:property name="servo_effort"    value="1.0"/>
   <xacro:property name="servo_velocity"  value="4.0"/>
-  <xacro:property name="servo_torque"    value="0.5"/>
-  <xacro:property name="servo_reduction" value="10.0"/>
+  <xacro:property name="servo_torque"    value="1.0"/>
+  <xacro:property name="servo_reduction" value="1.0"/>
   <xacro:property name="coxa_lower" value="-1.0"/>
   <xacro:property name="coxa_upper" value="1.0"/>
@@ -54,6 +54,6 @@
         <box size="0.02 0.01 0.03"/>
       </geometry>
-        <mass value="0.009"/>
-        <xacro:box_inertia m="0.009" x="0.02" y="0.01" z="0.03" />
+        <mass value="0.1"/>
+        <xacro:box_inertia m="0.1" x="0.02" y="0.01" z="0.03" />
     </inertial>
   </link>
@@ -96,6 +96,6 @@
         <box size="0.04 0.01 0.03"/>
       </geometry>
-        <mass value="0.001"/>
-        <xacro:box_inertia m="0.001" x="0.04" y="0.01" z="0.03" />
+        <mass value="0.1"/>
+        <xacro:box_inertia m="0.1" x="0.04" y="0.01" z="0.03" />
     </inertial>
   </link>
@@ -127,6 +127,6 @@
         <box size="0.02 0.01 0.03"/>
       </geometry>
-        <mass value="0.009"/>
-        <xacro:box_inertia m="0.009" x="0.02" y="0.01" z="0.03" />
+        <mass value="0.1"/>
+        <xacro:box_inertia m="0.1" x="0.02" y="0.01" z="0.03" />
     </inertial>
   </link>
@@ -169,6 +169,6 @@
         <box size="0.05 0.01 0.03"/>
       </geometry>
-        <mass value="0.002"/>
-        <xacro:box_inertia m="0.002" x="0.05" y="0.01" z="0.03" />
+        <mass value="0.2"/>
+        <xacro:box_inertia m="0.2" x="0.05" y="0.01" z="0.03" />
     </inertial>
   </link>
@@ -183,5 +183,5 @@
     <limit effort="${servo_effort}" velocity="${servo_velocity}" lower="-1.0" upper="1.0"/>
     <axis xyz="${side} 0 0"/>
-    <dynamics friction="0.7"/>
+    <!-- <dynamics friction="0.7"/> -->
   </joint>
   <transmission name="${name}_tibia_transmission">
@@ -216,6 +216,6 @@
         <box size="0.02 0.01 0.03"/>
       </geometry>
-        <mass value="0.009"/>
-        <xacro:box_inertia m="0.009" x="0.02" y="0.01" z="0.03" />
+        <mass value="0.1"/>
+        <xacro:box_inertia m="0.1" x="0.02" y="0.01" z="0.03" />
     </inertial>
   </link>
@@ -243,6 +243,6 @@
         <box size="0.1 0.005 0.005"/>
       </geometry>
-        <mass value="0.001"/>
-        <xacro:box_inertia m="0.001" x="0.1" y="0.005" z="0.005" />
+        <mass value="0.1"/>
+        <xacro:box_inertia m="0.1" x="0.1" y="0.005" z="0.005" />
     </inertial>
   </link>
@@ -281,10 +281,10 @@
           <sphere radius="0.005"/>
         </geometry>
-          <mass value="0.001"/>
-          <xacro:sphere_inertia m="0.001" r="0.005"/>
+          <mass value="0.1"/>
+          <xacro:sphere_inertia m="0.1" r="0.005"/>
       </inertial>
     </link>
     <gazebo reference="${name}_paw_link">
-      <!-- <gravity>true</gravity>
+      <gravity>true</gravity>
       <selfCollide>true</selfCollide>
       <mu1>100.0</mu1>
@@ -293,5 +293,5 @@
       <kd>1.0</kd>
       <fdir1>1 0 0</fdir1>
-      <maxContacts>1</maxContacts> -->
+      <maxContacts>1</maxContacts>
       <minDepth>0.0002</minDepth>
       <collision name="${name}__paw_link_collision">
@@ -303,23 +303,9 @@
         <surface>
           <friction>
-            <ode>
-              <mu>100000.0</mu>
-              <mu2>100000.0</mu2>
-            </ode>
             <torsional>
-              <coefficient>1000000</coefficient>
-              <use_patch_radius>true</use_patch_radius>
-              <surface_radius>0.005</surface_radius>
-              <patch_radius>0.005</patch_radius>
-            </torsional>
-          </friction>
-        </surface>
-        <!-- <surface>
-          <friction>
-            <torsional>
-                <coefficient>10</coefficient>
+                <coefficient>1000000</coefficient>
                 <use_patch_radius>true</use_patch_radius>
-                <surface_radius>0.1</surface_radius>
-                <patch_radius>0.1</patch_radius>
+                <surface_radius>0.005</surface_radius>
+                <patch_radius>0.005</patch_radius>
             </torsional>
           </friction>
@@ -328,5 +314,5 @@
             <elastic_modulus>1e8</elastic_modulus>
           </contact>
-        </surface> -->
+        </surface>
       </collision>
       <material>Gazebo/Red</material>
